Commit message: modify urdf

File: resources/robots/Ddogw/urdf/Ddogw.urdf (robot description, URDF)
Before this commit: robot Ddogw, 17 links, 16 joints
Joints:
- joint FL_foot_joint: limit effort=27 velocity=27 -> lower=-999999 upper=999999 effort=27 velocity=27
- joint FR_foot_joint: limit effort=27 velocity=27 -> lower=-999999 upper=999999 effort=27 velocity=27
- joint RL_foot_joint: limit effort=27 velocity=27 -> lower=-999999 upper=999999 effort=27 velocity=27
- joint RR_foot_joint: limit effort=27 velocity=27 -> lower=-999999 upper=999999 effort=27 velocity=27

Commit message: test but still stairs failed

File: resources/robots/Ddogw/urdf/Ddogw.urdf (robot description, URDF)
Before this commit: robot Ddogw, 17 links, 16 joints
Links:
- added link FL_foot_motor, mass 0.50; collision cylinder length=0.05 radius=0.03
- added link FR_foot_motor, mass 0.50; collision cylinder length=0.05 radius=0.03
- added link RL_foot_motor, mass 0.50; collision cylinder length=0.05 radius=0.03
- added link RR_foot_motor, mass 0.50; collision cylinder length=0.05 radius=0.03
- link FL_calf: mass 0.87 -> 0.37; geometry collision cylinder length=0.06 radius=0.015; visual mesh filename=../meshes/FL_CALF_Link.STL
- link FL_thigh: geometry collision cylinder length=0.10 radius=0.018; collision cylinder length=0.10 radius=0.03
- link FR_calf: mass 0.87 -> 0.37; geometry collision cylinder length=0.06 radius=0.015; visual mesh filename=../meshes/FR_CALF_Link.STL
- link FR_thigh: geometry collision cylinder length=0.10 radius=0.018; collision cylinder length=0.10 radius=0.03
- link RL_calf: mass 0.87 -> 0.37; geometry collision cylinder length=0.06 radius=0.015; visual mesh filename=../meshes/RL_CALF_Link.STL
- link RL_thigh: geometry collision cylinder length=0.10 radius=0.018; collision cylinder length=0.10 radius=0.03
- link RR_calf: mass 0.87 -> 0.37; geometry collision cylinder length=0.06 radius=0.015; visual mesh filename=../meshes/RR_CALF_Link.STL
- link RR_thigh: geometry collision cylinder length=0.10 radius=0.018; collision cylinder length=0.10 radius=0.03
Joints:
- added joint FL_foot_motor_joint: type fixed, parent FL_calf, child FL_foot_motor, origin xyz=0 -0.01 -0.219 rpy=0 0 0
- added joint FR_foot_motor_joint: type fixed, parent FR_calf, child FR_foot_motor, origin xyz=0 0.01 -0.219 rpy=0 0 0
- added joint RL_foot_motor_joint: type fixed, parent RL_calf, child RL_foot_motor, origin xyz=0 -0.01 -0.219 rpy=0 0 0
- added joint RR_foot_motor_joint: type fixed, parent RR_calf, child RR_foot_motor, origin xyz=0 0.01 -0.219 rpy=0 0 0
